Commit message: indentation, links on README 🧹️

File: desplate_xacro/sdf/inertial_box.sdf.xacro (robot description, xacro)
@@ -1,16 +1,16 @@
 <?xml version="1.0"?>
-<sdf xmlns:xacro="http://www.ros.org/wiki/xacro" >
-    <xacro:macro name="inertial_box" params="mass x y z">
-        <inertial>
-            <mass>${mass}</mass>
-            <inertia>
-              <ixx>${mass * (y*y+z*z) / 12.0}</ixx>
-              <ixy>0.0</ixy>
-              <ixz>0.0</ixz>
-              <iyy>${mass * (x*x+z*z) / 12.0}</iyy>
-              <iyz>0.0</iyz>
-              <izz>${mass * (x*x+y*y) / 12.0}</izz>
-            </inertia>
-        </inertial>
-    </xacro:macro>
+<sdf xmlns:xacro="http://www.ros.org/wiki/xacro">
+  <xacro:macro name="inertial_box" params="mass x y z">
+    <inertial>
+      <mass>${mass}</mass>
+      <inertia>
+        <ixx>${mass * (y*y+z*z) / 12.0}</ixx>
+        <ixy>0.0</ixy>
+        <ixz>0.0</ixz>
+        <iyy>${mass * (x*x+z*z) / 12.0}</iyy>
+        <iyz>0.0</iyz>
+        <izz>${mass * (x*x+y*y) / 12.0}</izz>
+      </inertia>
+    </inertial>
+  </xacro:macro>
 </sdf>

File: desplate_xacro/sdf/inertial_cylinder.sdf.xacro (robot description, xacro)
@@ -1,22 +1,22 @@
 <?xml version="1.0"?>
-<sdf xmlns:xacro="http://www.ros.org/wiki/xacro" >
-    <xacro:macro name="inertial_cylinder" params="mass radius length">
-        <xacro:property
-          name="xy"
-          value="${mass * (3 * radius * radius + length * length) / 12.0}"/>
-        <xacro:property
-          name="z"
-          value="${mass * radius * radius * 0.5}"/>
-        <inertial>
-            <mass>${mass}</mass>
-            <inertia>
-              <ixx>${xy}</ixx>
-              <ixy>0.0</ixy>
-              <ixz>0.0</ixz>
-              <iyy>${xy}</iyy>
-              <iyz>0.0</iyz>
-              <izz>${z}</izz>
-            </inertia>
-        </inertial>
-    </xacro:macro>
+<sdf xmlns:xacro="http://www.ros.org/wiki/xacro">
+  <xacro:macro name="inertial_cylinder" params="mass radius length">
+    <xacro:property
+      name="xy"
+      value="${mass * (3 * radius * radius + length * length) / 12.0}"/>
+    <xacro:property
+      name="z"
+      value="${mass * radius * radius * 0.5}"/>
+    <inertial>
+      <mass>${mass}</mass>
+      <inertia>
+        <ixx>${xy}</ixx>
+        <ixy>0.0</ixy>
+        <ixz>0.0</ixz>
+        <iyy>${xy}</iyy>
+        <iyz>0.0</iyz>
+        <izz>${z}</izz>
+      </inertia>
+    </inertial>
+  </xacro:macro>
 </sdf>

File: desplate_xacro/sdf/inertial_sphere.sdf.xacro (robot description, xacro)
@@ -1,19 +1,19 @@
 <?xml version="1.0"?>
-<sdf xmlns:xacro="http://www.ros.org/wiki/xacro" >
-    <xacro:macro name="inertial_sphere" params="mass radius">
-        <xacro:property
-          name="inertia"
-          value="${(2 * mass * radius * radius) / 5.0}"/>
-        <inertial>
-            <mass>${mass}</mass>
-            <inertia>
-              <ixx>${inertia}</ixx>
-              <ixy>0.0</ixy>
-              <ixz>0.0</ixz>
-              <iyy>${inertia}</iyy>
-              <iyz>0.0</iyz>
-              <izz>${inertia}</izz>
-            </inertia>
-        </inertial>
-    </xacro:macro>
+<sdf xmlns:xacro="http://www.ros.org/wiki/xacro">
+  <xacro:macro name="inertial_sphere" params="mass radius">
+    <xacro:property
+      name="inertia"
+      value="${(2 * mass * radius * radius) / 5.0}"/>
+    <inertial>
+      <mass>${mass}</mass>
+      <inertia>
+        <ixx>${inertia}</ixx>
+        <ixy>0.0</ixy>
+        <ixz>0.0</ixz>
+        <iyy>${inertia}</iyy>
+        <iyz>0.0</iyz>
+        <izz>${inertia}</izz>
+      </inertia>
+    </inertial>
+  </xacro:macro>
 </sdf>

File: desplate_xacro/sdf/vehicle.sdf.xacro (robot description, xacro)
@@ -1,4 +1,4 @@
 <?xml version="1.0"?>
-<sdf version="1.7" xmlns:xacro="http://www.ros.org/wiki/xacro">
+<sdf xmlns:xacro="http://www.ros.org/wiki/xacro" version="1.7">
   <model name="vehicle">
     <xacro:include filename="inertial_box.sdf.xacro"/>
@@ -7,63 +7,62 @@
     <xacro:include filename="wheel.sdf.xacro"/>
     <!-- Inputs -->
-    <xacro:property name="chassis_size_x" value="1.0" />
-    <xacro:property name="chassis_size_y" value="0.5" />
-    <xacro:property name="chassis_size_z" value="0.15" />
-    <xacro:property name="chassis_mass" value="1.0" />
-    <xacro:property name="wheel_radius" value="0.15" />
-    <xacro:property name="wheel_length" value="0.05" />
-    <xacro:property name="wheel_mass" value="0.5" />
-    <xacro:property name="caster_radius" value="0.1" />
-    <xacro:property name="caster_mass" value="0.0415553" />
+    <xacro:property name="chassis_size_x" value="1.0"/>
+    <xacro:property name="chassis_size_y" value="0.5"/>
+    <xacro:property name="chassis_size_z" value="0.15"/>
+    <xacro:property name="chassis_mass" value="1.0"/>
+    <xacro:property name="wheel_radius" value="0.15"/>
+    <xacro:property name="wheel_length" value="0.05"/>
+    <xacro:property name="wheel_mass" value="0.5"/>
+    <xacro:property name="caster_radius" value="0.1"/>
+    <xacro:property name="caster_mass" value="0.0415553"/>
     <!-- Calculated properties -->
-    <xacro:property name="wheel_offset_x" value="${chassis_size_x * 0.3}" />
-    <xacro:property name="wheel_offset_y" value="${(chassis_size_y + wheel_length) * 0.5}" />
-    <xacro:property name="wheel_offset_z" value="${-wheel_radius * 0.5}" />
-    <xacro:property name="caster_offset_x" value="${-chassis_size_x * 0.3}" />
-    <xacro:property name="caster_offset_y" value="0" />
-    <xacro:property name="caster_offset_z" value="${-(chassis_size_z + caster_radius) * 0.5}" />
+    <xacro:property name="wheel_offset_x" value="${chassis_size_x * 0.3}"/>
+    <xacro:property name="wheel_offset_y" value="${(chassis_size_y + wheel_length) * 0.5}"/>
+    <xacro:property name="wheel_offset_z" value="${-wheel_radius * 0.5}"/>
+    <xacro:property name="caster_offset_x" value="${-chassis_size_x * 0.3}"/>
+    <xacro:property name="caster_offset_y" value="0"/>
+    <xacro:property name="caster_offset_z" value="${-(chassis_size_z + caster_radius) * 0.5}"/>
     <xacro:macro name="material_macro" params="color_name">
-        <xacro:if value="${color_name == 'grey'}">
-          <xacro:property name="color" value="0.8 0.8 0.8 1"/>
-        </xacro:if>
-        <xacro:if value="${color_name == 'black'}">
-          <xacro:property name="color" value="0 0 0 1"/>
-        </xacro:if>
-        <material>
-          <diffuse>${color}</diffuse>
-          <specular>${color}</specular>
-          <ambient>${color}</ambient>
-        </material>
+      <xacro:if value="${color_name == 'grey'}">
+        <xacro:property name="color" value="0.8 0.8 0.8 1"/>
+      </xacro:if>
+      <xacro:if value="${color_name == 'black'}">
+        <xacro:property name="color" value="0 0 0 1"/>
+      </xacro:if>
+      <material>
+        <diffuse>${color}</diffuse>
+        <specular>${color}</specular>
+        <ambient>${color}</ambient>
+      </material>
     </xacro:macro>
     <link name="chassis">
-        <visual name="visual">
-            <geometry>
-                <box>
-                    <size>
-                      ${chassis_size_x}
-                      ${chassis_size_y}
-                      ${chassis_size_z}
-                    </size>
-                </box>
-            </geometry>
-            <xacro:material_macro
-              color_name="grey"/>
-        </visual>
-        <collision name="collision">
-            <geometry>
-                <box>
-                    <size>
-                      ${chassis_size_x}
-                      ${chassis_size_y}
-                      ${chassis_size_z}
-                    </size>
-                </box>
-            </geometry>
-        </collision>
-        <xacro:inertial_box
-          mass="${chassis_mass}"
-          x="${chassis_size_x}"
-          y="${chassis_size_y}"
-          z="${chassis_size_z}"/>
+      <visual name="visual">
+        <geometry>
+          <box>
+            <size>
+               ${chassis_size_x}
+               ${chassis_size_y}
+               ${chassis_size_z}
+             </size>
+          </box>
+        </geometry>
+        <xacro:material_macro color_name="grey"/>
+      </visual>
+      <collision name="collision">
+        <geometry>
+          <box>
+            <size>
+              ${chassis_size_x}
+              ${chassis_size_y}
+              ${chassis_size_z}
+            </size>
+          </box>
+        </geometry>
+      </collision>
+      <xacro:inertial_box
+        mass="${chassis_mass}"
+        x="${chassis_size_x}"
+        y="${chassis_size_y}"
+        z="${chassis_size_z}"/>
     </link>
     <xacro:wheel side="left"/>
@@ -72,9 +71,9 @@
     <!-- TODO(chapulina) Use ball - currently doesn't work with joint_state_publisher -->
     <joint name="caster_wheel_joint" type="fixed">
-        <parent>chassis</parent>
-        <child>caster_wheel</child>
+      <parent>chassis</parent>
+      <child>caster_wheel</child>
     </joint>
     <link name="caster_wheel">
-        <pose>
+      <pose>
           ${caster_offset_x}
           ${caster_offset_y}
@@ -82,24 +81,23 @@
           0 0 0
         </pose>
-        <visual name="visual">
-            <geometry>
-                <sphere>
-                  <radius>${caster_radius}</radius>
-                </sphere>
-            </geometry>
-            <xacro:material_macro
-              color_name="black"/>
-        </visual>
-        <collision name="collision">
-            <geometry>
-                <sphere>
-                  <radius>${caster_radius}</radius>
-                </sphere>
-            </geometry>
-        </collision>
-        <xacro:inertial_sphere
-          mass="${caster_mass}"
-          radius="${caster_radius}"/>
+      <visual name="visual">
+        <geometry>
+          <sphere>
+            <radius>${caster_radius}</radius>
+          </sphere>
+        </geometry>
+        <xacro:material_macro color_name="black"/>
+      </visual>
+      <collision name="collision">
+        <geometry>
+          <sphere>
+            <radius>${caster_radius}</radius>
+          </sphere>
+        </geometry>
+      </collision>
+      <xacro:inertial_sphere
+        mass="${caster_mass}"
+        radius="${caster_radius}"/>
     </link>
-</model>
+  </model>
 </sdf>

File: desplate_xacro/sdf/wheel.sdf.xacro (robot description, xacro)
@@ -1,4 +1,4 @@
 <?xml version="1.0"?>
-<sdf xmlns:xacro="http://www.ros.org/wiki/xacro" >
+<sdf xmlns:xacro="http://www.ros.org/wiki/xacro">
   <!-- Generates one of the actuated cylindrical wheels -->
   <xacro:macro name="wheel" params="side">
@@ -11,12 +11,12 @@
     <!-- TODO(chapulina) Use revolute - currently doesn't work with joint_state_publisher -->
     <joint name="${side}_wheel_joint" type="fixed">
-        <parent>chassis</parent>
-        <child>${side}_wheel</child>
-        <axis>
-          <xyz>0 0 1</xyz>
-        </axis>
+      <parent>chassis</parent>
+      <child>${side}_wheel</child>
+      <axis>
+        <xyz>0 0 1</xyz>
+      </axis>
     </joint>
     <link name="${side}_wheel">
-        <pose>
+      <pose>
           ${wheel_offset_x}
           ${offset_y}
@@ -26,26 +26,25 @@
           0
         </pose>
-        <visual name="visual">
-            <geometry>
-              <cylinder>
-                <radius>${wheel_radius}</radius>
-                <length>${wheel_length}</length>
-              </cylinder>
-            </geometry>
-            <xacro:material_macro
-              color_name="black"/>
-        </visual>
-        <collision name="collision">
-            <geometry>
-              <cylinder>
-                <radius>${wheel_radius}</radius>
-                <length>${wheel_length}</length>
-              </cylinder>
-            </geometry>
-        </collision>
-            <xacro:inertial_cylinder
-                mass="${wheel_mass}"
-                radius="${wheel_radius}"
-                length="${wheel_length}"/>
+      <visual name="visual">
+        <geometry>
+          <cylinder>
+            <radius>${wheel_radius}</radius>
+            <length>${wheel_length}</length>
+          </cylinder>
+        </geometry>
+        <xacro:material_macro color_name="black"/>
+      </visual>
+      <collision name="collision">
+        <geometry>
+          <cylinder>
+            <radius>${wheel_radius}</radius>
+            <length>${wheel_length}</length>
+          </cylinder>
+        </geometry>
+      </collision>
+      <xacro:inertial_cylinder
+        mass="${wheel_mass}"
+        radius="${wheel_radius}"
+        length="${wheel_length}"/>
     </link>
   </xacro:macro>

File: desplate_xacro/urdf/inertial_box.urdf.xacro (robot description, xacro)
@@ -1,15 +1,15 @@
 <?xml version="1.0"?>
-<robot xmlns:xacro="http://www.ros.org/wiki/xacro" >
-    <xacro:macro name="inertial_box" params="mass x y z">
-        <inertial>
-            <mass value="${mass}" />
-            <inertia
-              ixx="${mass * (y*y+z*z) / 12.0}"
-              ixy="0.0"
-              ixz="0.0"
-              iyy="${mass * (x*x+z*z) / 12.0}"
-              iyz="0.0"
-              izz="${mass * (x*x+y*y) / 12.0}" />
-        </inertial>
-    </xacro:macro>
+<robot xmlns:xacro="http://www.ros.org/wiki/xacro">
+  <xacro:macro name="inertial_box" params="mass x y z">
+    <inertial>
+      <mass value="${mass}" />
+      <inertia
+        ixx="${mass * (y*y+z*z) / 12.0}"
+        ixy="0.0"
+        ixz="0.0"
+        iyy="${mass * (x*x+z*z) / 12.0}"
+        iyz="0.0"
+        izz="${mass * (x*x+y*y) / 12.0}" />
+    </inertial>
+  </xacro:macro>
 </robot>

File: desplate_xacro/urdf/inertial_cylinder.urdf.xacro (robot description, xacro)
@@ -1,21 +1,21 @@
 <?xml version="1.0"?>
-<robot xmlns:xacro="http://www.ros.org/wiki/xacro" >
-    <xacro:macro name="inertial_cylinder" params="mass radius length">
-        <xacro:property
-          name="xy"
-          value="${mass * (3 * radius * radius + length * length) / 12.0}"/>
-        <xacro:property
-          name="z"
-          value="${mass * radius * radius * 0.5}"/>
-        <inertial>
-            <mass value="${mass}" />
-            <inertia
-              ixx="${xy}"
-              ixy="0.0"
-              ixz="0.0"
-              iyy="${xy}"
-              iyz="0.0"
-              izz="${z}" />
-        </inertial>
-    </xacro:macro>
+<robot xmlns:xacro="http://www.ros.org/wiki/xacro">
+  <xacro:macro name="inertial_cylinder" params="mass radius length">
+    <xacro:property
+      name="xy"
+      value="${mass * (3 * radius * radius + length * length) / 12.0}"/>
+    <xacro:property
+      name="z"
+      value="${mass * radius * radius * 0.5}"/>
+    <inertial>
+      <mass value="${mass}" />
+      <inertia
+        ixx="${xy}"
+        ixy="0.0"
+        ixz="0.0"
+        iyy="${xy}"
+        iyz="0.0"
+        izz="${z}" />
+    </inertial>
+  </xacro:macro>
 </robot>

File: desplate_xacro/urdf/inertial_sphere.urdf.xacro (robot description, xacro)
@@ -1,18 +1,18 @@
 <?xml version="1.0"?>
-<robot xmlns:xacro="http://www.ros.org/wiki/xacro" >
-    <xacro:macro name="inertial_sphere" params="mass radius">
-        <xacro:property
-          name="inertia"
-          value="${(2 * mass * radius * radius) / 5.0}"/>
-        <inertial>
-            <mass value="${mass}" />
-            <inertia
-              ixx="${inertia}"
-              ixy="0.0"
-              ixz="0.0"
-              iyy="${inertia}"
-              iyz="0.0"
-              izz="${inertia}" />
-        </inertial>
-    </xacro:macro>
+<robot xmlns:xacro="http://www.ros.org/wiki/xacro">
+  <xacro:macro name="inertial_sphere" params="mass radius">
+    <xacro:property
+      name="inertia"
+      value="${(2 * mass * radius * radius) / 5.0}"/>
+    <inertial>
+      <mass value="${mass}" />
+      <inertia
+        ixx="${inertia}"
+        ixy="0.0"
+        ixz="0.0"
+        iyy="${inertia}"
+        iyz="0.0"
+        izz="${inertia}" />
+    </inertial>
+  </xacro:macro>
 </robot>

File: desplate_xacro/urdf/vehicle.urdf.xacro (robot description, xacro)
@@ -1,72 +1,72 @@
 <?xml version="1.0"?>
 <robot xmlns:xacro="http://www.ros.org/wiki/xacro" name="vehicle">
-    <xacro:include filename="inertial_box.urdf.xacro"/>
-    <xacro:include filename="inertial_cylinder.urdf.xacro"/>
-    <xacro:include filename="inertial_sphere.urdf.xacro"/>
-    <xacro:include filename="wheel.urdf.xacro"/>
-    <!-- Inputs -->
-    <xacro:property name="chassis_size_x" value="1.0" />
-    <xacro:property name="chassis_size_y" value="0.5" />
-    <xacro:property name="chassis_size_z" value="0.15" />
-    <xacro:property name="chassis_mass" value="1.0" />
-    <xacro:property name="wheel_radius" value="0.15" />
-    <xacro:property name="wheel_length" value="0.05" />
-    <xacro:property name="wheel_mass" value="0.5" />
-    <xacro:property name="caster_radius" value="0.1" />
-    <xacro:property name="caster_mass" value="0.0415553" />
-    <!-- Calculated properties -->
-    <xacro:property name="wheel_x_offset" value="${chassis_size_x * 0.3}" />
-    <xacro:property name="wheel_y_offset" value="${(chassis_size_y + wheel_length) * 0.5}" />
-    <xacro:property name="wheel_z_offset" value="${-wheel_radius * 0.5}" />
-    <xacro:property name="caster_x_offset" value="${-chassis_size_x * 0.3}" />
-    <xacro:property name="caster_y_offset" value="0" />
-    <xacro:property name="caster_z_offset" value="${-(chassis_size_z + caster_radius) * 0.5}" />
-    <material name="grey">
-        <color rgba="0.8 0.8 0.8 1" />
-    </material>
-    <material name="black">
-        <color rgba="0 0 0 1"/>
-    </material>
-    <link name="chassis">
-        <visual>
-            <geometry>
-                <box size="${chassis_size_x} ${chassis_size_y} ${chassis_size_z}"/>
-            </geometry>
-            <material name="grey"/>
-        </visual>
-        <collision>
-            <geometry>
-                <box size="${chassis_size_x} ${chassis_size_y} ${chassis_size_z}"/>
-            </geometry>
-        </collision>
-        <xacro:inertial_box
-          mass="${chassis_mass}"
-          x="${chassis_size_x}"
-          y="${chassis_size_y}"
-          z="${chassis_size_z}"/>
-    </link>
-    <xacro:wheel side="left"/>
-    <xacro:wheel side="right"/>
-    <!-- caster -->
-    <joint name="caster_wheel_joint" type="fixed">
-        <parent link="chassis"/>
-        <child link="caster_wheel"/>
-        <origin xyz="${caster_x_offset} ${caster_y_offset} ${caster_z_offset}"/>
-    </joint>
-    <link name="caster_wheel">
-        <visual>
-            <geometry>
-                <sphere radius="${caster_radius}"/>
-            </geometry>
-            <material name="black"/>
-        </visual>
-        <collision>
-            <geometry>
-                <sphere radius="${caster_radius}"/>
-            </geometry>
-        </collision>
-        <xacro:inertial_sphere
-          mass="${caster_mass}"
-          radius="${caster_radius}"/>
-    </link>
+  <xacro:include filename="inertial_box.urdf.xacro"/>
+  <xacro:include filename="inertial_cylinder.urdf.xacro"/>
+  <xacro:include filename="inertial_sphere.urdf.xacro"/>
+  <xacro:include filename="wheel.urdf.xacro"/>
+  <!-- Inputs -->
+  <xacro:property name="chassis_size_x" value="1.0" />
+  <xacro:property name="chassis_size_y" value="0.5" />
+  <xacro:property name="chassis_size_z" value="0.15" />
+  <xacro:property name="chassis_mass" value="1.0" />
+  <xacro:property name="wheel_radius" value="0.15" />
+  <xacro:property name="wheel_length" value="0.05" />
+  <xacro:property name="wheel_mass" value="0.5" />
+  <xacro:property name="caster_radius" value="0.1" />
+  <xacro:property name="caster_mass" value="0.0415553" />
+  <!-- Calculated properties -->
+  <xacro:property name="wheel_x_offset" value="${chassis_size_x * 0.3}" />
+  <xacro:property name="wheel_y_offset" value="${(chassis_size_y + wheel_length) * 0.5}" />
+  <xacro:property name="wheel_z_offset" value="${-wheel_radius * 0.5}" />
+  <xacro:property name="caster_x_offset" value="${-chassis_size_x * 0.3}" />
+  <xacro:property name="caster_y_offset" value="0" />
+  <xacro:property name="caster_z_offset" value="${-(chassis_size_z + caster_radius) * 0.5}" />
+  <material name="grey">
+    <color rgba="0.8 0.8 0.8 1" />
+  </material>
+  <material name="black">
+    <color rgba="0 0 0 1"/>
+  </material>
+  <link name="chassis">
+    <visual>
+      <geometry>
+        <box size="${chassis_size_x} ${chassis_size_y} ${chassis_size_z}"/>
+      </geometry>
+      <material name="grey"/>
+    </visual>
+    <collision>
+      <geometry>
+        <box size="${chassis_size_x} ${chassis_size_y} ${chassis_size_z}"/>
+      </geometry>
+    </collision>
+    <xacro:inertial_box
+      mass="${chassis_mass}"
+      x="${chassis_size_x}"
+      y="${chassis_size_y}"
+      z="${chassis_size_z}"/>
+  </link>
+  <xacro:wheel side="left"/>
+  <xacro:wheel side="right"/>
+  <!-- caster -->
+  <joint name="caster_wheel_joint" type="fixed">
+    <parent link="chassis"/>
+    <child link="caster_wheel"/>
+    <origin xyz="${caster_x_offset} ${caster_y_offset} ${caster_z_offset}"/>
+  </joint>
+  <link name="caster_wheel">
+    <visual>
+      <geometry>
+        <sphere radius="${caster_radius}"/>
+      </geometry>
+      <material name="black"/>
+    </visual>
+    <collision>
+      <geometry>
+        <sphere radius="${caster_radius}"/>
+      </geometry>
+    </collision>
+    <xacro:inertial_sphere
+      mass="${caster_mass}"
+      radius="${caster_radius}"/>
+  </link>
 </robot>
